File: APRS-Tracker_KiCad/KiCad/APRS-Tracker_ArduinoProMini.kicad_pcb (KiCad board)
At the start: 2 copper layers, 70 x 55 mm, 23 parts, among them J1 Conn_01x03_Male, J2 Conn_01x05_Male, Q1 BS170, SW1 SW_Push, SW2 SW_SPDT, U1 TP4056, U2 MCP1700-3302E_TO92, U3 Arduino-Pro-Mini

Commit message: New file format
Other:
- net class Default removed
